File: batteries.sch (KiCad schematic (older format))
At the start: 23 parts, among them M2 Bilge Pump, SW1 BatterySwitch-12Both, SW2 Blue Sea 9003E, U1 BatteryCharger, U2 Blue Sea 7610, U3 PropaneGasDetector

Commit message: Many changes to original design
Parts:
- removed M2: Bilge Pump, symbol Motor:Motor_DC
- removed R1: Victron BMV-700, symbol Device:R_Shunt
- added F2-? (x3): 1A, symbol Device:Fuse
- added F3-1, F3-2, F3-3: 5A, symbol Device:Fuse
- added M1: Bilge Pump, symbol AvionicSchematic:Motor_DC
- added U4: VictronSmartShunt, symbol AvionicSchematic:VictronSmartShunt
- F1: value 300A -> 175A
- F2: value 175A -> 5A
- F2-1: value 15A -> 20A
Connections:
- net EngineGnd is gone; now on net DCOutGnd: BB2.1, BT1.2 (-), BT2.2 (-), BT3.2 (-)
- net DCOutGnd: now also ALT1.2 (-), BB2.3, BB2.4, BB2.5, BB2.6, F2-5.1, U1.4 (Bat1Neg), U1.6 (Bat2Neg), U1.8 (Bat3Neg), U3.1 (GND), M1.2 (-), U4.1 (Bat), U4.2 (Load)
- net at BT1.1 (+), BT2.1 (+), F1.2: now also F3-1.2, F3-2.2
- net BatTestStart: now reaches BT3.1 (+), F5.1, SW2.1 (Inp)
- net BatTestStart: now also F3-3.2
- net BatTestHouse: now reaches BB1.1, F1.1
- net BatTestHouse: now also BB1.2, BB1.3, BB1.4, BB1.5, BB1.6, F2-1.1, F2-2.1, F2-3.1, F2-4.1, F2.1, F3.1, F4.1, SW1.1
- net at U1.5 (Bat1Pos): now also F3-1.1
- net at U1.7 (Bat2Pos): now also F3-2.1
- net at F2.2: now also U4.4 (+B1); no longer U1.8 (Bat3Neg)
- net at U1.9 (Bat3Pos): now also F3-3.1
- net at F2-1.2: now also M1.1 (+)
- new net UTP: U4.3 (UTP)
- no-connect marks 0 -> 7
Other:
- note added: "Fuse Box\nATM Fuses"
- note added: "Switch Functions"
- moved on the sheet: F5, SW2, U1
