File: zephyr_schematic.sch (KiCad schematic (older format))
At the start: 0 parts

Commit message: Many changes to original design
Changed lines of the file:
@@
 $Descr USLetter 11000 8500
 encoding utf-8
-Sheet 1 2
+Sheet 1 3
 Title "Zephyr Electrical"
 Date ""
@@
 F0 "Batteries & Charging" 50
 F1 "batteries.sch" 50
+F2 "DCOutPos" U R 4000 3800 50
+F3 "DCOutGnd" U R 4000 3900 50
+F4 "Starter" U L 3000 4400 50
+F5 "EngineGnd" U L 3000 4300 50
+F6 "UTP" B R 4000 4375 50
 $EndSheet
-Text HLabel 3000 4075 2    50   UnSpc ~ 0
-DCOutPos
-Text HLabel 4000 3925 0    50   UnSpc ~ 0
-DCOutGnd
-Text HLabel 3000 3925 2    50   UnSpc ~ 0
-Starter
-Text HLabel 4000 4075 0    50   UnSpc ~ 0
-EngineGnd
+$Sheet
+S 4825 3700 1075 875
+U 60AAFAA5
+F0 "Main DC Panel" 50
+F1 "DC_house.sch" 50
+F2 "DCBatteryPos" I L 4825 3850 50
+F3 "DCBatteryNeg" I L 4825 3950 50
+F4 "UTP" B R 5900 4400 50
+$EndSheet
+Wire Wire Line
+	4000 3800 4425 3800
+Wire Wire Line
+	4425 3800 4425 3850
+Wire Wire Line
+	4425 3850 4825 3850
+Wire Wire Line
+	4000 3900 4425 3900
+Wire Wire Line
+	4425 3900 4425 3950
+Wire Wire Line
+	4425 3950 4825 3950
+Wire Wire Line
+	4000 4375 4400 4375
+Wire Wire Line
+	4400 4375 4400 4750
+Wire Wire Line
+	4400 4750 6025 4750
+Wire Wire Line
+	6025 4750 6025 4400
+Wire Wire Line
+	6025 4400 5900 4400
 $EndSCHEMATC
